File: projects/tiburon/esc_board.sch (EAGLE design)
At the start: 32 parts, among them J10 1X2-3.5MM, J11 1X2-3.5MM, J12 1X2-3.5MM, J7 1X2-3.5MM, J8 1X2-3.5MM, J9 1X2-3.5MM, Q10 BUZ11BH, Q11 BUZ11BH, Q12 BUZ11BH, Q7 BUZ11BH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

Commit message: added
Parts:
- added J1: (no value), SparkFun-Connectors:BATTERY_CONN_DEANS
Connections:
- net E16.8V: now also J1.+
- net GNDE: now also J1.-
Changed lines of the file:
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@@
 <part name="J11" library="adafruit" library_urn="urn:adsk.eagle:library:420" deviceset="1X2" device="-3.5MM" package3d_urn="urn:adsk.eagle:package:6240635/1"/>
 <part name="J12" library="adafruit" library_urn="urn:adsk.eagle:library:420" deviceset="1X2" device="-3.5MM" package3d_urn="urn:adsk.eagle:package:6240635/1"/>
+<part name="J1" library="SparkFun-Connectors" deviceset="BATTERY_CONN" device="_DEANS"/>
 </parts>
 <sheets>
@@
 <instance part="J11" gate="G$1" x="121.92" y="-55.88" smashed="yes"/>
 <instance part="J12" gate="G$1" x="167.64" y="-55.88" smashed="yes"/>
+<instance part="J1" gate="G$1" x="-76.2" y="45.72" smashed="yes">
+<attribute name="VALUE" x="-78.74" y="38.1" size="1.778" layer="96" font="vector"/>
+<attribute name="NAME" x="-78.74" y="49.022" size="1.778" layer="95" font="vector"/>
+</instance>
 </instances>
 <busses>
@@
 <label x="-73.66" y="-27.94" size="1.778" layer="95" rot="R180" xref="yes"/>
 </segment>
+<segment>
+<pinref part="J1" gate="G$1" pin="-"/>
+<wire x1="-68.58" y1="43.18" x2="-63.5" y2="43.18" width="0.1524" layer="91"/>
+<wire x1="-63.5" y1="43.18" x2="-63.5" y2="35.56" width="0.1524" layer="91"/>
+<label x="-63.5" y="35.56" size="1.778" layer="95" xref="yes"/>
+</segment>
 </net>
 <net name="N$2" class="0">
@@
 <pinref part="J12" gate="G$1" pin="1"/>
 </segment>
-</net>
+<segment>
+<pinref part="J1" gate="G$1" pin="+"/>
+<wire x1="-68.58" y1="45.72" x2="-63.5" y2="45.72" width="0.1524" layer="91"/>
+<wire x1="-63.5" y1="45.72" x2="-63.5" y2="53.34" width="0.1524" layer="91"/>
+<label x="-63.5" y="53.34" size="1.778" layer="95" xref="yes"/>
+</segment>
+</net>
