File: projects/tiburon/main_board.brd (EAGLE design)
At the start: 394.9 x 261.3 mm, 102 parts, among them IC2 7812, J6 1X2-3.5MM, M2 ARDUINO-NANO-3.0#ISP, Q1 MOSFET-PCHANNELFQP27P06, Q2 MOSFET-PCHANNELFQP27P06, Q3 BC548

Commit message: added
Parts:
- removed C2, C3: 10nF, SparkFun-Capacitors:CAP-PTH-10MM
- removed J2: (no value), SparkFun-Connectors:DEANS
- added C10, C9: (no value), rcl:C025-025X050
- added JP24: (no value), adafruit:1X03
- added JP25, JP26: Extra Reed, pinhead:1X02
- C1, C4, C5, C6, C7, C8: value 10nF -> (none); device SparkFun-Capacitors:CAP-PTH-10MM -> rcl:C025-025X050
- moved C8 401.3 mm to (179.1, 115.6), turned to 90 degrees
- moved JP23 388.0 mm to (162.6, 119.4)
- moved R34 331.2 mm to (165.1, 82.5), turned to 270 degrees
- moved JP18 327.3 mm to (195.6, 43.2), turned to 180 degrees
- moved R33 326.7 mm to (162.6, 82.5), turned to 270 degrees
- moved C7 325.4 mm to (162.6, -3.81), turned to 180 degrees
- moved JP20 325.1 mm to (195.6, 34.3), turned to 90 degrees
- moved R30 315.1 mm to (171.4, 104.1), turned to 270 degrees
- moved LED4 308.1 mm to (167.6, 91.4), turned to 90 degrees
- moved JP21 287.6 mm to (69.8, 80.0), turned to 270 degrees
- moved LED6 284.0 mm to (116.8, 81.3)
- moved Q3 282.2 mm to (124.5, 78.7), turned to 270 degrees
- moved R32 274.9 mm to (110.5, 80.0), turned to 90 degrees
- moved IC5 272.6 mm to (191.8, -6.35)
- moved IC2 271.5 mm to (119.4, -10.2), turned to 180 degrees
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Connections:
- net INA_1 renamed N$73
- net INB_1 renamed N$24
- net INC_1 renamed N$68
- removed net EAD2: JP10.11, M2.J1.5, R9.2
- removed net INA_2: JP22.8, U$6.6, U$7.8
- removed net INB_2: JP22.10, U$6.8, U$7.9
- removed net INC_2: JP22.12, U$6.10, U$7.10
- removed net N$110: JP22.9, U$6.7
- removed net N$112: JP22.11, U$6.9
- removed net N$114: JP22.13, U$6.11
- removed net N$24 (its old number): JP1.1, U$7.18
- removed net N$47 (its old number): JP8.4, NUC.J2.4
- removed net N$58: JP8.5, NUC.J2.5
- removed net N$59: JP8.6, NUC.J2.6
- removed net N$63: JP8.14, NUC.J2.14
- removed net N$65: LED3.A, R21.1
- removed net N$69: JP9.4, NUC.J1.4
- removed net N$71: JP18.2, JP9.12, NUC.J1.12
- removed net N$72: JP9.13, NUC.J1.13
- removed net N$73 (its old number): JP9.14, NUC.J1.14
- removed net N$84 (its old number): JP10.10, M2.J1.6
- removed net N$85: JP10.12, M2.J1.4
- new net ED3: JP10.10, LED1.A, M2.J1.6
- new net N$1: JP10.11, M2.J1.5
- new net N$14: LED3.A, R21.2
- new net N$15: JP2.3, R10.2
- new net N$20: JP22.12, U$6.10
- new net N$34: JP1.2, U$7.13
- new net N$35: JP22.13, U$6.11, U$7.10
- new net N$39: JP1.4, U$7.14
- new net N$43: JP1.10, U$7.18
- new net N$45: JP18.2, JP9.13, NUC.J1.13
- new net N$46: JP25.2, JP9.14, NUC.J1.14
- new net N$49: JP22.11, U$6.9, U$7.9
- new net N$61: JP22.9, U$6.7, U$7.8
- net DR1_IN: now also JP9.9, NUC.J1.9; no longer JP9.6, NUC.J1.6
- net DR2_IN: now also JP9.10, NUC.J1.10; no longer JP9.7, NUC.J1.7
- net E16.8V: now also JP1.9, R19.2; no longer JP1.4, U$3.IN+
- net EN: now also JP1.3, U$7.15; no longer JP1.8
- net ENLED: now also JP9.5, NUC.J1.5
- net GNDE: now also C10.2, C8.2, JP1.7, JP10.12, JP11.2, JP24.3, M2.J1.4, M2.J2.2, R30.1, R9.1, U$7.19; no longer C2.2, C3.2, J2.-, LED1.K, LED4.K
- net GNDN: now also C9.2, JP17.2, JP25.1, JP26.1, JP8.2, JP9.4, NUC.J1.4, NUC.J2.2; no longer C8.2, JP17.1
- net GR1_IN: now also JP9.8, NUC.J1.8; no longer JP9.10, NUC.J1.10
- net GR2_IN: now also JP9.7, NUC.J1.7; no longer JP9.11, NUC.J1.11
- net N$10: now also JP2.8; no longer JP2.6
- net N$100: now also C7.1; no longer C1.1
- net N$102: now also Q1.2; no longer Q1.3
- net N$11: now also JP2.10; no longer JP2.4
- net N$16: now also JP2.5, R11.2; no longer JP2.9, R10.2
- net N$17: now also LED4.K, R30.2; no longer JP2.7, R11.2
- net N$18: now also JP2.9; no longer JP2.5
- net N$19: now also JP2.7; no longer JP2.3
- net N$22: now also JP22.10, U$6.8; no longer J2.+, Q2.2, R19.2
- net N$23: now also C10.1; no longer C2.1
- net N$25: now also Q2.2, U$3.IN+; no longer JP1.3, U$7.17
- net N$27: now also JP17.1, JP8.14, NUC.J2.14, R33.1, R34.1; no longer JP1.5, U$7.16
- net N$28: now also D2.C, JP21.1, JP8.4, NUC.J2.4; no longer JP1.7, U$7.14
- net N$29: now also JP11.4, JP23.1, JP24.2, JP3.2, JP4.2, JP5.2, M2.J2.4; no longer JP1.9, U$7.13
- net N$30: now also JP8.10, NUC.J2.10, R12.1, R16.2; no longer JP1.10, U$7.12
- net N$32: now also JP22.8, U$6.6; no longer D2.C, JP21.1
- net N$33: now also JP1.1, U$7.12; no longer JP1.2, U$7.19
- net N$36: now also C9.1, Q1.3; no longer C7.1, Q1.2
- net N$37: now also C1.1; no longer C8.1
- net N$40: now also JP1.6, U$7.16; no longer JP11.2, M2.J2.2
- net N$41: now also JP1.8, U$7.17; no longer LED4.A, R30.1
- net N$55: now also JP8.9, NUC.J2.9, R13.1, R17.2; no longer JP8.2, NUC.J2.2
- net N$64: now also R21.1; no longer R21.2
- net N$7: now also LED1.K, R9.2; no longer LED1.A, R9.1
- net N$8: now also JP2.4; no longer JP2.10
- net N$89: now also LED4.A; no longer R30.2
- net N$9: now also JP2.6; no longer JP2.8
- net N12V: now also JP26.2
- net N6V: now also C4.1; no longer C6.1
- net NA0: now also JP8.5, NUC.J2.5; no longer JP8.12, NUC.J2.12, R13.1, R17.2
- net NA1: now also JP8.6, NUC.J2.6; no longer JP8.11, NUC.J2.11, R12.1, R16.2
- net NA2: now also JP8.11, NUC.J2.11; no longer JP8.10, NUC.J2.10
- net NA3: now also JP8.12, NUC.J2.12; no longer JP8.9, NUC.J2.9
- net NTSOP: now also JP9.6, NUC.J1.6; no longer JP9.5, NUC.J1.5
- net TMP1: now also JP24.1; no longer JP5.2
- net TMP2: now also JP5.1; no longer JP4.2
- net TMP3: now also JP4.1; no longer JP3.2
- net TMP4: now also JP3.1
- net TP1_IN: now also JP9.11, NUC.J1.11; no longer JP9.8, NUC.J1.8
- net TP2_IN: now also JP9.12, NUC.J1.12; no longer JP9.9, NUC.J1.9
- net VCCE: now also C8.1; no longer C3.1, JP11.4, JP23.1, JP3.1, JP4.1, JP5.1, M2.J2.4
- net VCCN: now also C6.1; no longer C4.1, JP17.2, R33.1, R34.1
Routing:
- net GNDN: track 0.00 -> 701.4 mm
- net GNDE: track 0.00 -> 341.0 mm
- net VCCE: track 0.00 -> 208.7 mm, vias 0 -> 3
- net VCCN: track 0.00 -> 182.6 mm, vias 0 -> 2
- net N$100: track 0.00 -> 170.7 mm
- net N12V: track 0.00 -> 170.2 mm
- net N$28: track 0.00 -> 141.8 mm
- net E16.8V: track 0.00 -> 74.5 mm
- net N$102: track 0.00 -> 68.5 mm
- net N$23: track 0.00 -> 63.2 mm
- net EN: track 0.00 -> 61.1 mm
- net N$68: track 0.00 -> 56.4 mm
- net DR1: track 0.00 -> 56.3 mm, vias 0 -> 2
- net N$2: track 0.00 -> 52.9 mm
- net N$101: track 0.00 -> 52.9 mm
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- added copper zone on layer 1, net MOTOR
Other:
- board size 394.9 x 261.3 mm -> 137.1 x 141.9 mm
