File: projects/tiburon/main_board.sch (EAGLE design)
At the start: 102 parts, among them IC2 7812, J6 1X2-3.5MM, M2 ARDUINO-NANO-3.0#ISP, Q1 MOSFET-PCHANNELFQP27P06, Q2 MOSFET-PCHANNELFQP27P06, Q3 BC548

Commit message: added
Parts:
- removed C2, C3: 10nF, SparkFun-Capacitors:10NF-PTH-10MM-10000V-1-%
- removed J2: (no value), SparkFun-Connectors:BATTERY_CONN_DEANS
- added C10, C9: (no value), rcl:C-EU025-025X050
- added JP24: (no value), adafruit:PINHD-1X3
- added JP25, JP26: Extra Reed, pinhead:PINHD-1X2
- C1, C4, C5, C6, C7, C8: value 10nF -> (none); device SparkFun-Capacitors:10NF-PTH-10MM-10000V-1-% -> rcl:C-EU025-025X050
Connections:
- net INA_1 renamed N$73
- net INB_1 renamed N$24
- net INC_1 renamed N$68
- removed net EAD2: JP10.11, M2.D2, R9.2
- removed net INA_2: JP22.8, U$6.6, U$7.INA_2
- removed net INB_2: JP22.10, U$6.8, U$7.INB_2
- removed net INC_2: JP22.12, U$6.10, U$7.INC_2
- removed net N$110: JP22.9, U$6.7
- removed net N$112: JP22.11, U$6.9
- removed net N$114: JP22.13, U$6.11
- removed net N$24 (its old number): JP1.1, U$7.OUTA_1
- removed net N$47 (its old number): JP8.4, NUC.5V
- removed net N$58: JP8.5, NUC.A7
- removed net N$59: JP8.6, NUC.A6
- removed net N$63: JP8.14, NUC.3V3
- removed net N$65: LED3.A, R21.1
- removed net N$69: JP9.4, NUC.GND.1
- removed net N$71: JP18.2, JP9.12, NUC.D9
- removed net N$72: JP9.13, NUC.D10
- removed net N$73 (its old number): JP9.14, NUC.D11/MOSI
- removed net N$84 (its old number): JP10.10, M2.D3
- removed net N$85: JP10.12, M2.GND.1
- new net ED3: JP10.10, LED1.A, M2.D3
- new net N$1: JP10.11, M2.D2
- new net N$14: LED3.A, R21.2
- new net N$15: JP2.3, R10.2
- new net N$20: JP22.12, U$6.10
- new net N$34: JP1.2, U$7.OUTB_2
- new net N$35: JP22.13, U$6.11, U$7.INC_2
- new net N$39: JP1.4, U$7.OUTA_2
- new net N$43: JP1.10, U$7.OUTA_1
- new net N$45: JP18.2, JP9.13, NUC.D10
- new net N$46: JP25.2, JP9.14, NUC.D11/MOSI
- new net N$49: JP22.11, U$6.9, U$7.INB_2
- new net N$61: JP22.9, U$6.7, U$7.INA_2
- net DR1_IN: now also JP9.9, NUC.D6; no longer JP9.6, NUC.D3
- net DR2_IN: now also JP9.10, NUC.D7; no longer JP9.7, NUC.D4
- net E16.8V: now also JP1.9, R19.2; no longer JP1.4, U$3.IN+
- net EN: now also JP1.3, U$7.KILL(1); no longer JP1.8
- net ENLED: now also JP9.5, NUC.D2
- net GNDE: now also C10.2, C8.2, JP1.7, JP10.12, JP11.2, JP24.3, M2.GND.1, M2.GND.2, R30.1, R9.1, U$7.GND2(1); no longer C2.2, C3.2, J2.-, LED1.C, LED4.C
- net GNDN: now also C9.2, JP17.2, JP25.1, JP26.1, JP8.2, JP9.4, NUC.GND.1, NUC.GND.2; no longer C8.2, JP17.1
- net GR1_IN: now also JP9.8, NUC.D5; no longer JP9.10, NUC.D7
- net GR2_IN: now also JP9.7, NUC.D4; no longer JP9.11, NUC.D8
- net N$10: now also JP2.8; no longer JP2.6
- net N$100: now also C7.1; no longer C1.1
- net N$102: now also Q1.D; no longer Q1.S
- net N$11: now also JP2.10; no longer JP2.4
- net N$16: now also JP2.5, R11.2; no longer JP2.9, R10.2
- net N$17: now also LED4.C, R30.2; no longer JP2.7, R11.2
- net N$18: now also JP2.9; no longer JP2.5
- net N$19: now also JP2.7; no longer JP2.3
- net N$22: now also JP22.10, U$6.8; no longer J2.+, Q2.D, R19.2
- net N$23: now also C10.1; no longer C2.1
- net N$25: now also Q2.D, U$3.IN+; no longer JP1.3, U$7.OUTB_1
- net N$27: now also JP17.1, JP8.14, NUC.3V3, R33.1, R34.1; no longer JP1.5, U$7.OUTC_1
- net N$28: now also D2.C, JP21.1, JP8.4, NUC.5V; no longer JP1.7, U$7.OUTA_2
- net N$29: now also JP11.4, JP23.1, JP24.2, JP3.2, JP4.2, JP5.2, M2.5V; no longer JP1.9, U$7.OUTB_2
- net N$30: now also JP8.10, NUC.A2, R12.1, R16.2; no longer JP1.10, U$7.OUTC_2
- net N$32: now also JP22.8, U$6.6; no longer D2.C, JP21.1
- net N$33: now also JP1.1, U$7.OUTC_2; no longer JP1.2, U$7.GND2(1)
- net N$36: now also C9.1, Q1.S; no longer C7.1, Q1.D
- net N$37: now also C1.1; no longer C8.1
- net N$40: now also JP1.6, U$7.OUTC_1; no longer JP11.2, M2.GND.2
- net N$41: now also JP1.8, U$7.OUTB_1; no longer LED4.A, R30.1
- net N$55: now also JP8.9, NUC.A3, R13.1, R17.2; no longer JP8.2, NUC.GND.2
- net N$64: now also R21.1; no longer R21.2
- net N$7: now also LED1.C, R9.2; no longer LED1.A, R9.1
- net N$8: now also JP2.4; no longer JP2.10
- net N$89: now also LED4.A; no longer R30.2
- net N$9: now also JP2.6; no longer JP2.8
- net N12V: now also JP26.2
- net N6V: now also C4.1; no longer C6.1
- net NA0: now also JP8.5, NUC.A7; no longer JP8.12, NUC.A0, R13.1, R17.2
- net NA1: now also JP8.6, NUC.A6; no longer JP8.11, NUC.A1, R12.1, R16.2
- net NA2: now also JP8.11, NUC.A1; no longer JP8.10, NUC.A2
- net NA3: now also JP8.12, NUC.A0; no longer JP8.9, NUC.A3
- net NTSOP: now also JP9.6, NUC.D3; no longer JP9.5, NUC.D2
- net TMP1: now also JP24.1; no longer JP5.2
- net TMP2: now also JP5.1; no longer JP4.2
- net TMP3: now also JP4.1; no longer JP3.2
- net TMP4: now also JP3.1
- net TP1_IN: now also JP9.11, NUC.D8; no longer JP9.8, NUC.D5
- net TP2_IN: now also JP9.12, NUC.D9; no longer JP9.9, NUC.D6
- net VCCE: now also C8.1; no longer C3.1, JP11.4, JP23.1, JP3.1, JP4.1, JP5.1, M2.5V
- net VCCN: now also C6.1; no longer C4.1, JP17.2, R33.1, R34.1
Other:
- moved on the sheet: C1, C4, C6, C7, C8, JP1, JP18, JP3, JP4, LED3, LED4, Q1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
